File: ma12070p_amp_v1.kicad_pcb (KiCad board)
At the start: 2 copper layers, 81 parts, among them J2 Screw_Terminal_01x04, J3 Screw_Terminal_01x02, U1 MA12070P, U2 TPS62175DQC

Commit message: small updates to pcb
Parts:
- CLIP LED: renamed from CLIP_LED_0
- moved RCLK1 0.85 mm to (129.1, 96.3)
- moved RIN0B1 0.36 mm to (125.8, 88.4)
- moved RIN1B1 0.35 mm to (126.1, 96.2)
- renumbered RCLIP_LED_0 to CLIP, RCLIP_ERROR_0 to ERR, ERROR_LED_0 to E_LED
Routing:
- net /VDD: track 318.8 -> 314.0 mm
- net /PVDD: track 199.9 -> 195.7 mm
- net GND: track 57.2 -> 54.3 mm, vias 136 -> 134
- net Net-(CAPIN0A1-Pad1): track 26.6 -> 24.1 mm
- net AD1: track 13.8 -> 14.6 mm, vias 2 -> 1
- net CLK: track 29.6 -> 29.1 mm
- net AD0: vias 2 -> 1

Commit message: change
Parts:
- removed CAPIN0A1, CAPIN0B1, CAPIN1A1, CAPIN1B1, CCDC0, CCREF0, CFDC0, CGD0, CGD0N1, CGD1, CGD1N1, COUTBUCK1, CPVDD0B0, CPVDD0B1, CPVDD0B3, CPVDD1B0, CVGDC0: 1uF, Capacitor_SMD:C_1206_3216Metric
- removed CF0A0, CF0A1, CF0B0, CF0B1, CF1A0, CF1A1, CF1B0, CF1B1: 10uF, Capacitor_SMD:C_1206_3216Metric
- removed CFGD0, CGD0N0, CGD1N0, COUTBUCK2, CPVDD0A0, CPVDD1A0: 0.1uF, Capacitor_SMD:C_1206_3216Metric
- removed CIN0: 22nF, Capacitor_SMD:C_1206_3216Metric
- removed CLIP, ERR: 2k, Resistor_SMD:R_1206_3216Metric
- removed CLIP LED: LED, LED_SMD:LED_1206_3216Metric
- removed COUTBUCK0: 22uF, Capacitor_THT:CP_Radial_D6.3mm_P2.50mm
- removed CSUP1, CSUP2: 330uF/35V, Capacitor_THT:CP_Radial_D10.0mm_P5.00mm
- removed E_LED: LED, LED_SMD:LED_1206_3216Metric
- removed J2: Screw_Terminal_01x04, TerminalBlock_Phoenix:TerminalBlock_Phoenix_MKDS-1,5-4_1x04_P5.00mm_Horizontal
- removed J3: Screw_Terminal_01x02, TerminalBlock_Phoenix:TerminalBlock_Phoenix_MKDS-1,5-2_1x02_P5.00mm_Horizontal
- removed LBUCK0: SRN4026-100M, Inductor_SMD:L_Bourns-SRN4018
- removed LSUP0: Ferrite 2743019447, Inductor_SMD:L_2010_5025Metric_Pad1.52x2.65mm_HandSolder
- removed PAUDIO1, PCTRL1: Conn_01x05, Connector_PinHeader_2.54mm:PinHeader_1x05_P2.54mm_Vertical
- removed RB_FB1: 2M, Resistor_SMD:R_1206_3216Metric
- removed RB_FB2: 383k, Resistor_SMD:R_1206_3216Metric
- removed RB_PG0: 100k, Resistor_SMD:R_1206_3216Metric
- removed RCLK1, RENABLE1, RIN0B1, RIN1B1, RMUTE1: R, Resistor_SMD:R_1206_3216Metric
- removed RPVDD1: 0.1R, Resistor_SMD:R_1206_3216Metric
- added C12: 1uF, Capacitor_TH_TDK:C_Rect_L7.3_W4.5_P5.0, F.Cu at (193.0, 75.0)
- added C13: 0.47uF, Capacitor_TH_TDK:C_Rect_L7.3_W4.5_P5.0, F.Cu at (193.0, 81.0)
- added C14: 0.1uF, Capacitor_SMD:C_1206_3216Metric_Pad1.33x1.80mm_HandSolder, F.Cu at (144.6, 55.9)
- added C15: 4,7uF, Capacitor_SMD:C_1206_3216Metric_Pad1.33x1.80mm_HandSolder, F.Cu at (133.7, 59.0)
- added C16: 0.1uF, Capacitor_SMD:C_1206_3216Metric_Pad1.33x1.80mm_HandSolder, F.Cu at (133.7, 62.0)
- added C17: 10uF, Capacitor_SMD:C_1206_3216Metric_Pad1.33x1.80mm_HandSolder, F.Cu at (144.0, 76.0)
- added C18: 10uF, Capacitor_SMD:C_1206_3216Metric_Pad1.33x1.80mm_HandSolder, F.Cu at (144.0, 79.0)
- added C19: 1uF, Capacitor_SMD:C_1206_3216Metric_Pad1.33x1.80mm_HandSolder, F.Cu at (133.7, 52.0)
- added C2: 100uF, Capacitor_THT:CP_Radial_D10.0mm_P5.00mm, F.Cu at (151.6, 67.2)
- added C20: 22uF, Capacitor_SMD:C_1206_3216Metric_Pad1.33x1.80mm_HandSolder, F.Cu at (133.7, 55.0)
- added C21: 10uF, Capacitor_SMD:C_1206_3216Metric_Pad1.33x1.80mm_HandSolder, F.Cu at (155.9, 100.0)
- added C22: 10uF, Capacitor_SMD:C_1206_3216Metric_Pad1.33x1.80mm_HandSolder, F.Cu at (155.9, 97.0)
- added C23: 1uF, Capacitor_TH_TDK:C_Rect_L7.3_W4.5_P5.0, F.Cu at (193.0, 101.0)
- added C24: 0.47uF, Capacitor_TH_TDK:C_Rect_L7.3_W4.5_P5.0, F.Cu at (193.0, 95.0)
- added C25: 10uF, Capacitor_SMD:C_1206_3216Metric_Pad1.33x1.80mm_HandSolder, F.Cu at (144.0, 100.0)
- added C26: 10uF, Capacitor_SMD:C_1206_3216Metric_Pad1.33x1.80mm_HandSolder, F.Cu at (144.0, 97.0)
- added C27: 1uF, Capacitor_TH_TDK:C_Rect_L7.3_W4.5_P5.0, F.Cu at (193.0, 114.0)
- added C28: 0.47uF, Capacitor_TH_TDK:C_Rect_L7.3_W4.5_P5.0, F.Cu at (193.0, 108.0)
- added C29: 1uF, Capacitor_SMD:C_1206_3216Metric_Pad1.33x1.80mm_HandSolder, F.Cu at (162.0, 97.0)
- added C30: 1uF, Capacitor_SMD:C_1206_3216Metric_Pad1.33x1.80mm_HandSolder, F.Cu at (162.0, 100.0)
- added C31: 0.1uF, Capacitor_SMD:C_1206_3216Metric_Pad1.33x1.80mm_HandSolder, F.Cu at (162.0, 103.0)
- added C32: 22uF, Capacitor_SMD:C_1206_3216Metric_Pad1.33x1.80mm_HandSolder, F.Cu at (133.7, 65.2)
- added C33: 22uF, Capacitor_SMD:C_1206_3216Metric_Pad1.33x1.80mm_HandSolder, F.Cu at (133.8, 68.2)
- added C34: 1uF, Capacitor_SMD:C_1206_3216Metric_Pad1.33x1.80mm_HandSolder, F.Cu at (162.0, 88.0)
- added C35: 1uF, Capacitor_SMD:C_1206_3216Metric_Pad1.33x1.80mm_HandSolder, F.Cu at (162.0, 85.0)
- added C36: 0.1uF, Capacitor_SMD:C_1206_3216Metric_Pad1.33x1.80mm_HandSolder, F.Cu at (162.0, 82.0)
- added C37: 1uF, Capacitor_SMD:C_1206_3216Metric_Pad1.33x1.80mm_HandSolder, F.Cu at (162.0, 94.0)
- added C38: 1uF, Capacitor_SMD:C_1206_3216Metric_Pad1.33x1.80mm_HandSolder, F.Cu at (162.0, 79.0)
- added C39: 1uF, Capacitor_SMD:C_1206_3216Metric_Pad1.33x1.80mm_HandSolder, F.Cu at (162.0, 91.0)
- added C40: 0.1uF, Capacitor_SMD:C_1206_3216Metric_Pad1.33x1.80mm_HandSolder, F.Cu at (162.0, 76.0)
- added C41: 1uF, Capacitor_SMD:C_1206_3216Metric_Pad1.33x1.80mm_HandSolder, F.Cu at (138.2, 79.0)
- added C42: 1uF, Capacitor_SMD:C_1206_3216Metric_Pad1.33x1.80mm_HandSolder, F.Cu at (158.4, 122.0)
- added C43: 1uF, Capacitor_SMD:C_1206_3216Metric_Pad1.33x1.80mm_HandSolder, F.Cu at (138.2, 82.0)
- added C44: 1uF, Capacitor_SMD:C_1206_3216Metric_Pad1.33x1.80mm_HandSolder, F.Cu at (138.2, 85.0)
- added C45: 1uF, Capacitor_SMD:C_1206_3216Metric_Pad1.33x1.80mm_HandSolder, F.Cu at (138.2, 91.0)
- added C46: 1uF, Capacitor_SMD:C_1206_3216Metric_Pad1.33x1.80mm_HandSolder, F.Cu at (138.2, 88.0)
- added C6: 1uF, Capacitor_SMD:C_1206_3216Metric_Pad1.33x1.80mm_HandSolder, F.Cu at (150.0, 79.0)
- added C8: 1uF, Capacitor_TH_TDK:C_Rect_L7.3_W4.5_P5.0, F.Cu at (193.0, 62.0)
- added CIN2: 0.022uF, Capacitor_SMD:C_1206_3216Metric_Pad1.33x1.80mm_HandSolder, F.Cu at (125.2, 59.5)
- added CONN1: Screw_Terminal_01x02, TerminalBlock_Phoenix:TerminalBlock_Phoenix_MKDS-1,5-2_1x02_P5.00mm_Horizontal, F.Cu at (116.5, 69.8)
- added CONN2: Screw_Terminal_01x04, TerminalBlock_Phoenix:TerminalBlock_Phoenix_MKDS-1,5-4_1x04_P5.00mm_Horizontal, F.Cu at (208.7, 80.5)
- added CONN3: Conn_01x05, Connector_PinHeader_2.54mm:PinHeader_1x05_P2.54mm_Vertical, F.Cu at (120.2, 99.2)
- added CONN4: Conn_01x05, Connector_PinHeader_2.54mm:PinHeader_1x05_P2.54mm_Vertical, F.Cu at (120.2, 82.4)
- added JP5: SolderJumper_3_Open, Jumper:SolderJumper-3_P1.3mm_Open_Pad1.0x1.5mm, F.Cu at (132.0, 95.2)
- added JP6: SolderJumper_2_Open, Jumper:SolderJumper-2_P1.3mm_Open_Pad1.0x1.5mm, F.Cu at (132.2, 84.2)
- added JP7: SolderJumper_2_Open, Jumper:SolderJumper-2_P1.3mm_Open_Pad1.0x1.5mm, F.Cu at (138.2, 104.5)
- added JP8: SolderJumper_2_Open, Jumper:SolderJumper-2_P1.3mm_Open_Pad1.0x1.5mm, F.Cu at (138.2, 101.5)
- added JP9: SolderJumper_3_Open, Jumper:SolderJumper-3_P1.3mm_Open_Pad1.0x1.5mm, F.Cu at (132.0, 99.2)
- added L1: 47, Inductor_SMD:L_2010_5025Metric_Pad1.52x2.65mm_HandSolder, F.Cu at (124.4, 63.0)
- added L6: 6.8uH, Inductor_TH_Bourns:L_Radia_Zylinder_D9.0_P5.0, F.Cu at (178.0, 108.0)
- added LED1: LED, LED_SMD:LED_1206_3216Metric_Pad1.42x1.75mm_HandSolder, F.Cu at (164.4, 55.0)
- added LED2: LED, LED_SMD:LED_1206_3216Metric_Pad1.42x1.75mm_HandSolder, F.Cu at (164.4, 52.0)
- added R5: 3.6, Resistor_SMD:R_1206_3216Metric_Pad1.30x1.75mm_HandSolder, F.Cu at (186.0, 97.0)
- added R6: 2k, Resistor_SMD:R_1206_3216Metric_Pad1.30x1.75mm_HandSolder, F.Cu at (158.4, 55.0)
- added R7: 3.6, Resistor_SMD:R_1206_3216Metric_Pad1.30x1.75mm_HandSolder, F.Cu at (186.0, 110.0)
- added R8: 2k, Resistor_SMD:R_1206_3216Metric_Pad1.30x1.75mm_HandSolder, F.Cu at (158.4, 52.0)
- C1: value 0.47uF -> 100uF; footprint Capacitor_THT:C_Rect_L7.2mm_W4.5mm_P5.00mm_FKS2_FKP2_MKS2_MKP2 -> Capacitor_THT:CP_Radial_D10.0mm_P5.00mm
- C10: value 1uF -> 10uF; footprint Capacitor_THT:C_Rect_L13.0mm_W5.0mm_P10.00mm_FKS3_FKP3_MKS4 -> Capacitor_SMD:C_1206_3216Metric_Pad1.33x1.80mm_HandSolder
- C11: value 0.47uF -> 10uF; footprint Capacitor_THT:C_Rect_L7.2mm_W4.5mm_P5.00mm_FKS2_FKP2_MKS2_MKP2 -> Capacitor_SMD:C_1206_3216Metric_Pad1.33x1.80mm_HandSolder
- C3: footprint Capacitor_THT:C_Rect_L13.0mm_W5.0mm_P10.00mm_FKS3_FKP3_MKS4 -> Capacitor_SMD:C_1206_3216Metric_Pad1.33x1.80mm_HandSolder
- C4: value 1uF -> 0.1uF; footprint Capacitor_THT:C_Rect_L13.0mm_W5.0mm_P10.00mm_FKS3_FKP3_MKS4 -> Capacitor_SMD:C_1206_3216Metric_Pad1.33x1.80mm_HandSolder
- C5: value 0.47uF -> 0.1uF; footprint Capacitor_THT:C_Rect_L7.2mm_W4.5mm_P5.00mm_FKS2_FKP2_MKS2_MKP2 -> Capacitor_SMD:C_1206_3216Metric_Pad1.33x1.80mm_HandSolder
- C7: value 0.47uF -> 1uF; footprint Capacitor_THT:C_Rect_L7.2mm_W4.5mm_P5.00mm_FKS2_FKP2_MKS2_MKP2 -> Capacitor_SMD:C_1206_3216Metric_Pad1.33x1.80mm_HandSolder
- C9: value 1uF -> 0.47uF; footprint Capacitor_THT:C_Rect_L13.0mm_W5.0mm_P10.00mm_FKS3_FKP3_MKS4 -> Capacitor_TH_TDK:C_Rect_L7.3_W4.5_P5.0
- CIN1: value 22nF -> 0.022uF; footprint Capacitor_SMD:C_1206_3216Metric -> Capacitor_SMD:C_1206_3216Metric_Pad1.33x1.80mm_HandSolder
- JP1, JP3: value Jumper_3_Open -> SolderJumper_3_Open; footprint Connector_PinHeader_2.54mm:PinHeader_1x03_P2.54mm_Vertical -> Jumper:SolderJumper-3_P1.3mm_Open_Pad1.0x1.5mm
- JP2, JP4: value Jumper_3_Open -> SolderJumper_2_Open; footprint Connector_PinHeader_2.54mm:PinHeader_1x03_P2.54mm_Vertical -> Jumper:SolderJumper-2_P1.3mm_Open_Pad1.0x1.5mm
- L2, L4, L5: value 3.3uH -> 6.8uH; footprint Inductor_SMD:L_Bourns_SRP1245A -> Inductor_TH_Bourns:L_Radia_Zylinder_D9.0_P5.0
- L3: value 3.3uH -> 10uH; footprint Inductor_SMD:L_Bourns_SRP1245A -> Inductor_TH_Bourns:RLB0712-100KL
- R1: value 3.6 -> 0.1R; footprint Resistor_SMD:R_1206_3216Metric -> Resistor_SMD:R_1206_3216Metric_Pad1.30x1.75mm_HandSolder
- R2, R4: footprint Resistor_SMD:R_1206_3216Metric -> Resistor_SMD:R_1206_3216Metric_Pad1.30x1.75mm_HandSolder
- R3: value 3.6 -> 4.7k; footprint Resistor_SMD:R_1206_3216Metric -> Resistor_SMD:R_1206_3216Metric_Pad1.30x1.75mm_HandSolder
- U1: value MA12070P -> MAX16956AUBD/V+; footprint Package_DFN_QFN:QFN-64-1EP_9x9mm_P0.5mm_EP5.45x5.45mm -> max_16956:MAX16956AUBD&slash_V&plus_
- U2: value TPS62175DQC -> MA12070P; footprint Package_SON:WSON-10-1EP_2x3mm_P0.5mm_EP0.84x2.4mm_ThermalVias -> Package_DFN_QFN:QFN-64-1EP_9x9mm_P0.5mm_EP5.45x5.45mm
- moved R3 83.9 mm to (133.8, 48.8), turned to 0 degrees
- moved R1 76.5 mm to (117.4, 63.2), turned to 0 degrees
- moved C7 58.9 mm to (138.2, 76.0), turned to 180 degrees
- moved C10 57.4 mm to (156.0, 76.0), turned to 0 degrees
- moved C1 55.2 mm to (151.6, 108.5), turned to 0 degrees
- moved C3 55.1 mm to (150.0, 97.0), turned to 180 degrees
- moved C11 54.2 mm to (156.0, 79.0), turned to 0 degrees
- moved JP2 52.1 mm to (132.8, 104.5), turned to 0 degrees
- moved C4 49.5 mm to (150.0, 76.0), turned to 180 degrees
- moved U1 47.8 mm to (142.2, 51.9), turned to 180 degrees
- moved L3 43.5 mm to (146.1, 62.0)
- moved C5 43.2 mm to (150.0, 100.0), turned to 180 degrees
- moved R4 37.0 mm to (186.0, 79.0)
- moved U2 34.4 mm to (150.0, 88.0), turned to -90 degrees
- moved C9 32.4 mm to (193.0, 68.0), turned to 180 degrees
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Connections:
- C1 pad 1: GND -> PVDD
- C1 pad 2: Net-(C1-Pad2) -> GND
- C10 pad 2: GND -> Net-(C10-Pad2)
- C11 pad 1: Net-(C11-Pad1) -> Net-(C10-Pad1)
- C11 pad 2: GND -> Net-(C10-Pad2)
- C3 pad 1: GND -> PVDD
- C3 pad 2: Net-(C3-Pad2) -> GND
- C4 pad 1: Net-(C4-Pad1) -> PVDD
- C5 pad 1: Net-(C5-Pad1) -> PVDD
- C7 pad 1: GND -> VDD
- C7 pad 2: Net-(C7-Pad2) -> GND
- CIN1 pad 2: /PVDD -> Net-(CIN1-Pad2)
- JP1 pad 1: GND -> Buck_5V
- JP1 pad 2: AD1 -> VDD
- JP1 pad 3: /VDD -> IC_5V
- JP2 pad 1: /BUCK_5V -> GND
- JP2 pad 2: /VDD -> ENABLE
- JP3 pad 2: CLKM/S -> CLKMS
- JP3 pad 3: /VDD -> VDD
- JP4 pad 1: GND -> VDD
- JP4 pad 2: AD0 -> MUTE
- L2 pad 1: Net-(C1-Pad2) -> Net-(C9-Pad2)
- L3 pad 1: Net-(C5-Pad1) -> Net-(C14-Pad2)
- L3 pad 2: OUT0A -> IC_5V
- L4 pad 1: Net-(C7-Pad2) -> Net-(C13-Pad1)
- L4 pad 2: OUT1A -> OUT0A
- L5 pad 1: Net-(C11-Pad1) -> Net-(C24-Pad2)
- L5 pad 2: OUT1B -> OUT1A
- R1 pad 1: Net-(C1-Pad2) -> Net-(CONN1-Pad1)
- R1 pad 2: Net-(C3-Pad2) -> Net-(CIN1-Pad2)
- R2 pad 1: Net-(C4-Pad1) -> Net-(C9-Pad2)
- R2 pad 2: Net-(C5-Pad1) -> Net-(C8-Pad1)
- R3 pad 1: Net-(C7-Pad2) -> VDD
- R3 pad 2: Net-(C9-Pad2) -> Net-(R3-Pad2)
- R4 pad 1: Net-(C10-Pad1) -> Net-(C12-Pad1)
- R4 pad 2: Net-(C11-Pad1) -> Net-(C13-Pad1)
- U1 pad 1: GND -> Net-(C14-Pad1)
- U1 pad 10: OUT0B -> PVDD
- U1 pad 2: GND -> PVDD
- U1 pad 3: Net-(CF0A0-Pad2) -> Net-(C14-Pad2)
- U1 pad 4: OUT0A -> GND
- U1 pad 5: OUT0A -> GND
- U1 pad 6: Net-(CF0A0-Pad1) -> Net-(R3-Pad2)
- U1 pad 7: /PVDD -> Net-(C19-Pad1)
- U1 pad 8: /PVDD -> Net-(C19-Pad1)
- U1 pad 9: Net-(CF0B0-Pad1) -> IC_5V
- U2 pad 10: /BUCK_5V -> OUT0B
- U2 pad 11: GND -> OUT0B
- U2 pad 2: /PVDD -> GND
- U2 pad 3: /PVDD -> Net-(C10-Pad2)
- U2 pad 4: GND -> OUT0A
- U2 pad 5: Net-(RB_FB1-Pad1) -> OUT0A
- U2 pad 6: GND -> Net-(C10-Pad1)
- U2 pad 7: Net-(RB_PG0-Pad1) -> PVDD
- U2 pad 8: /BUCK_5V -> PVDD
Routing:
- net /VDD: track 314.0 -> 0.00 mm, vias 2 -> 0
- net VDD: track 0.00 -> 248.8 mm, vias 0 -> 8
- net PVDD: track 0.00 -> 200.4 mm, vias 0 -> 7
- net /PVDD: track 195.7 -> 0.00 mm, vias 8 -> 0
- net /CLIP: track 43.9 -> 0.00 mm, vias 2 -> 0
- net /ERROR: track 43.2 -> 0.00 mm, vias 2 -> 0
- net ERR: track 0.00 -> 37.0 mm, vias 0 -> 2
- net Net-(C11-Pad1): track 36.6 -> 0.00 mm
- net Net-(C45-Pad1): track 0.00 -> 36.5 mm, vias 0 -> 2
- net /BUCK_5V: track 36.2 -> 0.00 mm
- net Net-(C1-Pad2): track 36.0 -> 0.00 mm
- net Net-(C28-Pad1): track 0.00 -> 35.5 mm
- net GND: track 54.3 -> 89.5 mm, vias 134 -> 74
- net CLIP: track 0.00 -> 33.5 mm, vias 0 -> 2
- net Net-(C24-Pad2): track 0.00 -> 30.1 mm
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Other:
- board outline added: 105 x 85 mm

Commit message: new
Parts:
- U1: value MAX16956AUBD/V+ -> MAX16956
- moved C12 2.50 mm to (190.5, 75.0)
- moved C13 2.50 mm to (190.5, 81.0)
- moved C23 2.50 mm to (190.5, 101.0)
- moved C24 2.50 mm to (195.5, 95.0)
- moved C27 2.50 mm to (190.5, 114.0)
- moved C28 2.50 mm to (190.5, 108.0)
- moved C9 2.50 mm to (195.5, 68.0)
- moved C8 2.45 mm to (190.6, 62.0)
Other:
- board text added: "+"
- board text added: "OUT 0"
- board text added: "OUT 1"

Commit message: update again
Parts:
- AMP OUT: renamed from CONN2
- V IN: renamed from CONN1
- renumbered LED1 to CLIP, LED2 to ERROR, CONN4 to PAUDIO, CONN3 to PCTRL
Routing:
- net GND: track 89.5 -> 97.7 mm, vias 74 -> 76
Other:
- board text added: "ENABLE"
- board text added: "GND"
- board text added: "IN 0A"
- board text added: "IN 0B"
- board text added: "IN 1A"
- board text added: "IN 1B"
- board text added: "MUTE"
- board text added: "SDA"
- board text added: "SDL"

Commit message: V0.1
Parts:
- CONN1: renamed from V IN
- CONN2: renamed from AMP OUT
- U1: value MAX16956 -> MAX16956AUBD/V+
- moved C42 26.8 mm to (168.0, 97.0)
- moved C31 6.71 mm to (168.0, 100.0)
- moved H1 5.84 mm to (205.0, 119.0)
- moved JP1 5.52 mm to (134.0, 65.0), turned to 0 degrees
- moved H4 5.38 mm to (205.0, 49.0)
- moved CONN2 5.00 mm to (203.7, 80.5)
- moved H3 3.02 mm to (115.0, 119.0)
- moved C32 2.75 mm to (133.7, 68.0)
- moved C33 2.75 mm to (133.8, 71.0)
- moved H2 1.98 mm to (115.0, 49.0)
- moved C1 0.52 mm to (151.5, 109.0)
- renumbered PCTRL to CONN3, PAUDIO to CONN4, CLIP to LED1, ERROR to LED2
Connections:
- C42 pad 1: unconnected-(C42-Pad1) -> VDD
- C42 pad 2: unconnected-(C42-Pad2) -> GND
Routing:
- net VDD: track 248.8 -> 237.5 mm, vias 8 -> 9
- net GND: track 97.7 -> 107.4 mm
- net Net-(C29-Pad1): track 16.0 -> 21.6 mm
- net Net-(C9-Pad2): track 35.6 -> 30.6 mm
- net Net-(C28-Pad1): track 35.5 -> 30.5 mm
- net Net-(C24-Pad2): track 30.1 -> 25.1 mm
- net Net-(C13-Pad1): track 30.1 -> 25.1 mm
- net Net-(C14-Pad2): track 12.7 -> 15.5 mm
- net PVDD: track 200.4 -> 199.8 mm
Other:
- board size 105 x 85 mm -> 100 x 80 mm
- board text added: "By Fabian M"
- board text added: "IN0A/BCLK"
- board text added: "IN0B/WS"
- board text added: "IN1A/SD0"
- board text added: "IN1B/MCLK"
- board text added: "ma12070p AMP V0.1"
- board text removed: "IN 0A"
- board text removed: "IN 0B"
- board text removed: "IN 1A"
- board text removed: "IN 1B"

Commit message: finished DRC
Parts:
- R1: footprint Resistor_SMD:R_1206_3216Metric_Pad1.30x1.75mm_HandSolder -> Resistor_SMD:R_2512_6332Metric_Pad1.40x3.35mm_HandSolder
- moved R1 1.43 mm to (116.0, 63.0)
- moved CIN2 1.00 mm to (125.2, 58.5)
Connections:
- net Buck_5V renamed Ext_supply_5V
- U2 pad 65: (no net) -> GND
Routing:
- net GND: track 107.4 -> 23.4 mm, vias 76 -> 73
- net OUT1A: track 31.2 -> 26.3 mm
- net OUT1B: track 42.1 -> 37.1 mm
- net OUT0B: track 42.3 -> 37.4 mm
- net OUT0A: track 31.1 -> 26.2 mm
- net PVDD: track 199.8 -> 203.2 mm
- net VDD: track 237.5 -> 235.5 mm
- net Net-(C29-Pad1): track 21.6 -> 20.1 mm
- net Net-(CONN1-Pad1): track 7.12 -> 8.17 mm
- net Net-(C34-Pad2): track 10.3 -> 9.59 mm
- net Net-(C29-Pad2): track 13.4 -> 12.7 mm
- net SDA: track 32.2 -> 31.6 mm
- net Net-(CIN1-Pad2): track 7.53 -> 6.97 mm
- net Net-(C39-Pad1): track 7.48 -> 6.91 mm
- net Net-(C34-Pad1): track 6.17 -> 5.66 mm
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Other:
- board size 100 x 80 mm -> 100.4 x 80.4 mm

Commit message: minor Changes Vias
Routing:
- net GND: vias 73 -> 91
