File: ma12070p_amp_v1.kicad_sch (KiCad schematic)
At the start: 81 parts, among them J2 Screw_Terminal_01x04, J3 Screw_Terminal_01x02, U1 MA12070P, U2 TPS62175DQC

Commit message: update
Parts:
- CAPIN0A1, CAPIN0B1, CAPIN1A1, CAPIN1B1, CGD0N1, CGD1, CGD1N1: footprint Capacitor_SMD:C_1206_3216Metric -> Capacitor_SMD:C_0603_1608Metric
- CCDC1: renamed from CCDC0; footprint Capacitor_SMD:C_1206_3216Metric -> Capacitor_SMD:C_0603_1608Metric
- CCREF1: renamed from CCREF0; footprint Capacitor_SMD:C_1206_3216Metric -> Capacitor_SMD:C_0603_1608Metric
- CF0A1: renamed from CF0A0; footprint Capacitor_SMD:C_1206_3216Metric -> Capacitor_SMD:C_0603_1608Metric
- CF0A2: renamed from CF0A1; footprint Capacitor_SMD:C_1206_3216Metric -> Capacitor_SMD:C_0603_1608Metric
- CF0B1: renamed from CF0B0; footprint Capacitor_SMD:C_1206_3216Metric -> Capacitor_SMD:C_0603_1608Metric
- CF0B2: renamed from CF0B1; footprint Capacitor_SMD:C_1206_3216Metric -> Capacitor_SMD:C_0603_1608Metric
- CF1A1: renamed from CF1A0; footprint Capacitor_SMD:C_1206_3216Metric -> Capacitor_SMD:C_0603_1608Metric
- CF1A2: renamed from CF1A1; footprint Capacitor_SMD:C_1206_3216Metric -> Capacitor_SMD:C_0603_1608Metric
- CF1B1: renamed from CF1B0; footprint Capacitor_SMD:C_1206_3216Metric -> Capacitor_SMD:C_0603_1608Metric
- CF1B2: renamed from CF1B1; footprint Capacitor_SMD:C_1206_3216Metric -> Capacitor_SMD:C_0603_1608Metric
- CFDC1: renamed from CFDC0; footprint Capacitor_SMD:C_1206_3216Metric -> Capacitor_SMD:C_0603_1608Metric
- CFGD1: renamed from CFGD0; footprint Capacitor_SMD:C_1206_3216Metric -> Capacitor_SMD:C_0603_1608Metric
- CGD0N2: renamed from CGD0N0; footprint Capacitor_SMD:C_1206_3216Metric -> Capacitor_SMD:C_0603_1608Metric
- CGD1N2: renamed from CGD1N0; footprint Capacitor_SMD:C_1206_3216Metric -> Capacitor_SMD:C_0603_1608Metric
- CGD2: renamed from CGD0; footprint Capacitor_SMD:C_1206_3216Metric -> Capacitor_SMD:C_0603_1608Metric
- CIN1: renamed from CIN0; footprint Capacitor_SMD:C_1206_3216Metric -> Capacitor_SMD:C_0603_1608Metric
- CIN2: renamed from CIN1; footprint Capacitor_SMD:C_1206_3216Metric -> Capacitor_SMD:C_0603_1608Metric
- CPVDD0B2: renamed from CPVDD0B1; footprint Capacitor_SMD:C_1206_3216Metric -> Capacitor_SMD:C_0603_1608Metric
- CPVDD0B3: renamed from CPVDD0B0; footprint Capacitor_SMD:C_1206_3216Metric -> Capacitor_SMD:C_0603_1608Metric
- CPVDD1B1: renamed from CPVDD1B0; footprint Capacitor_SMD:C_1206_3216Metric -> Capacitor_SMD:C_0603_1608Metric
- R1, R2, R3, R4, RB_FB1, RB_FB2: footprint Resistor_SMD:R_1206_3216Metric -> Resistor_SMD:R_0603_1608Metric
- RB_PG1: renamed from RB_PG0; footprint Resistor_SMD:R_1206_3216Metric -> Resistor_SMD:R_0603_1608Metric
- renumbered C3 to C1, C4 to C2, C9 to C3, C10 to C4, C1 to C5, C5 to C6, C11 to C8, CLIP_LED_0 to CLIP_LED_1, COUTBUCK0 to COUTBUCK2, COUTBUCK2 to COUTBUCK3, CPVDD0A0 to CPVDD0A1, CPVDD0B3 to CPVDD0B1, CPVDD1A0 to CPVDD1A1, CVGDC0 to CVGDC1, ERROR_LED_0 to ERROR_LED_1, J3 to J1, JP2 to JP1, JP3 to JP2, JP4 to JP3, JP1 to JP4, L2 to L1, L3 to L2, L4 to L3, L5 to L4, LBUCK0 to LBUCK1, LSUP0 to LSUP1, RCLIP_ERROR_0 to RCLIP_ERROR_1, RCLIP_LED_0 to RCLIP_LED_1, U2 to U1, U1 to U2

Commit message: Revert "Merge branch 'main' of https://github.com/fabianmuehlberger/ma12070p_amp_kicad"
This reverts commit afd773a9720c15933af275e3fcdef7eeb23b86f2, reversing
changes made to a492eb96612e67492a35cba3f1296495fc6c8237.
Parts:
- removed C3, C4: 1uF, Capacitor_THT:C_Rect_L13.0mm_W5.0mm_P10.00mm_FKS3_FKP3_MKS4, symbol Device:C
- removed C7, C8: 0.47uF, Capacitor_THT:C_Rect_L7.2mm_W4.5mm_P5.00mm_FKS2_FKP2_MKS2_MKP2, symbol Device:C
- removed COUTBUCK2: 22uF, Capacitor_THT:CP_Radial_D6.3mm_P2.50mm, symbol Device:CP
- removed CPVDD0B1: 1uF, Capacitor_SMD:C_1206_3216Metric, symbol Device:C
- removed JP1, JP2, JP3, JP4: Jumper_3_Open, Connector_PinHeader_2.54mm:PinHeader_1x03_P2.54mm_Vertical, symbol Jumper:Jumper_3_Open
- removed L4: 3.3uH, Inductor_SMD:L_Bourns_SRP1245A, symbol Device:L
- removed LBUCK1: SRN4026-100M, Inductor_SMD:L_Bourns-SRN4018, symbol Device:L
- removed R4: 3.6, Resistor_SMD:R_0603_1608Metric, symbol Device:R
- removed RB_FB1: 2M, Resistor_SMD:R_0603_1608Metric, symbol Device:R
- removed RB_FB2: 383k, Resistor_SMD:R_0603_1608Metric, symbol Device:R
- removed RB_PG1: 100k, Resistor_SMD:R_0603_1608Metric, symbol Device:R
- removed RCLK1, RENABLE1, RIN0B1, RIN1B1, RMUTE1: R, Resistor_SMD:R_1206_3216Metric, symbol Device:R
- removed U1: TPS62175DQC, Package_SON:WSON-10-1EP_2x3mm_P0.5mm_EP0.84x2.4mm_ThermalVias, symbol Regulator_Switching:TPS62175DQC
- added C14, C16: 0.1uF, Capacitor_SMD:C_1206_3216Metric_Pad1.33x1.80mm_HandSolder, symbol Device:C
- added C15: 4,7uF, Capacitor_SMD:C_1206_3216Metric_Pad1.33x1.80mm_HandSolder, symbol Device:C
- added C19, C42: 1uF, Capacitor_SMD:C_1206_3216Metric_Pad1.33x1.80mm_HandSolder, symbol Device:C
- added C20: 22uF, Capacitor_SMD:C_1206_3216Metric_Pad1.33x1.80mm_HandSolder, symbol Device:C
- added C23, C27: 1uF, Capacitor_TH_TDK:C_Rect_L7.3_W4.5_P5.0, symbol Device:C
- added C24, C28: 0.47uF, Capacitor_TH_TDK:C_Rect_L7.3_W4.5_P5.0, symbol Device:C
- added JP1, JP3, JP5, JP9: SolderJumper_3_Open, Jumper:SolderJumper-3_P1.3mm_Open_Pad1.0x1.5mm, symbol Jumper:SolderJumper_3_Open
- added JP2, JP4, JP6, JP7, JP8: SolderJumper_2_Open, Jumper:SolderJumper-2_P1.3mm_Open_Pad1.0x1.5mm, symbol Jumper:SolderJumper_2_Open
- added L5, L6: 6.8uH, Inductor_TH_Bourns:L_Radia_Zylinder_D9.0_P5.0, symbol Device:L
- added R5, R7: 3.6, Resistor_SMD:R_1206_3216Metric_Pad1.30x1.75mm_HandSolder, symbol Device:R
- added U1: MAX16956AUBD/V+, max_16956:MAX16956AUBD&slash_V&plus_, symbol max_16956:MAX16956AUBD/V+
- C1: renamed from CSUP1; value 330uF/35V -> 100uF; DigikeyRef (none) -> UFG1V101MPM; infineonRef (none) -> CSUP1; property_1 (none) -> 35V; property_2 (none) -> UWT
- C10: renamed from CF0A1; footprint Capacitor_SMD:C_0603_1608Metric -> Capacitor_SMD:C_1206_3216Metric_Pad1.33x1.80mm_HandSolder; infineonRef (none) -> CF0A0; property_1 (none) -> X5R; property_2 (none) -> 25V
- C11: renamed from CF0A2; footprint Capacitor_SMD:C_0603_1608Metric -> Capacitor_SMD:C_1206_3216Metric_Pad1.33x1.80mm_HandSolder; infineonRef (none) -> CF0A1; property_1 (none) -> X5R; property_2 (none) -> 25V
- C12: renamed from C2; footprint Capacitor_THT:C_Rect_L13.0mm_W5.0mm_P10.00mm_FKS3_FKP3_MKS4 -> Capacitor_TH_TDK:C_Rect_L7.3_W4.5_P5.0; infineonRef (none) -> C0B0; property_1 (none) -> L13.0xW5.0
- C13: renamed from C6; footprint Capacitor_THT:C_Rect_L7.2mm_W4.5mm_P5.00mm_FKS2_FKP2_MKS2_MKP2 -> Capacitor_TH_TDK:C_Rect_L7.3_W4.5_P5.0; infineonRef (none) -> C0A1; property_1 (none) -> L7.2xW4.5
- C17: renamed from CF0B1; footprint Capacitor_SMD:C_0603_1608Metric -> Capacitor_SMD:C_1206_3216Metric_Pad1.33x1.80mm_HandSolder; infineonRef (none) -> CF0B0; property_1 (none) -> X5R; property_2 (none) -> 25V
- C18: renamed from CF0B2; footprint Capacitor_SMD:C_0603_1608Metric -> Capacitor_SMD:C_1206_3216Metric_Pad1.33x1.80mm_HandSolder; infineonRef (none) -> CF0B1; property_1 (none) -> X5R; property_2 (none) -> 25V
- C2: renamed from CSUP2; value 330uF/35V -> 100uF; DigikeyRef (none) -> UFG1V101MPM; infineonRef (none) -> CSUP2; property_1 (none) -> 35V; property_2 (none) -> UWT
- C21: renamed from CF1A1; footprint Capacitor_SMD:C_0603_1608Metric -> Capacitor_SMD:C_1206_3216Metric_Pad1.33x1.80mm_HandSolder; infineonRef (none) -> CF1A0; property_1 (none) -> X5R; property_2 (none) -> 25V
- C22: renamed from CF1A2; footprint Capacitor_SMD:C_0603_1608Metric -> Capacitor_SMD:C_1206_3216Metric_Pad1.33x1.80mm_HandSolder; infineonRef (none) -> CF1A1; property_1 (none) -> X5R; property_2 (none) -> 25V
- C25: renamed from CF1B1; footprint Capacitor_SMD:C_0603_1608Metric -> Capacitor_SMD:C_1206_3216Metric_Pad1.33x1.80mm_HandSolder; infineonRef (none) -> CF1B0; property_1 (none) -> X5R; property_2 (none) -> 25V
- C26: renamed from CF1B2; footprint Capacitor_SMD:C_0603_1608Metric -> Capacitor_SMD:C_1206_3216Metric_Pad1.33x1.80mm_HandSolder; infineonRef (none) -> CF1B1; property_1 (none) -> X5R; property_2 (none) -> 25V
- C29: renamed from CGD1; footprint Capacitor_SMD:C_0603_1608Metric -> Capacitor_SMD:C_1206_3216Metric_Pad1.33x1.80mm_HandSolder; infineonRef (none) -> CGD0; property_1 (none) -> X7R; property_2 (none) -> 25V
- C3: renamed from CPVDD0B3; footprint Capacitor_SMD:C_0603_1608Metric -> Capacitor_SMD:C_1206_3216Metric_Pad1.33x1.80mm_HandSolder; infineonRef (none) -> CPVDD0B; property_1 (none) -> X5R; property_2 (none) -> 50V
- C30: renamed from CGD1N1; footprint Capacitor_SMD:C_0603_1608Metric -> Capacitor_SMD:C_1206_3216Metric_Pad1.33x1.80mm_HandSolder; infineonRef (none) -> CGD1N1; property_1 (none) -> X5R; property_2 (none) -> 50V
- C31: renamed from CGD1N2; footprint Capacitor_SMD:C_0603_1608Metric -> Capacitor_SMD:C_1206_3216Metric_Pad1.33x1.80mm_HandSolder; infineonRef (none) -> CGD1N0; property_1 (none) -> X7R; property_2 (none) -> 50V
- C32: renamed from COUTBUCK1; value 1uF -> 22uF; footprint Capacitor_SMD:C_1206_3216Metric -> Capacitor_SMD:C_1206_3216Metric_Pad1.33x1.80mm_HandSolder; infineonRef (none) -> COUNTBUCK0; property_2 (none) -> 50V
- C33: renamed from COUTBUCK3; value 0.1uF -> 22uF; footprint Capacitor_SMD:C_1206_3216Metric -> Capacitor_SMD:C_1206_3216Metric_Pad1.33x1.80mm_HandSolder; infineonRef (none) -> COUNTBUCK1; property_2 (none) -> 50V
- C34: renamed from CFDC1; footprint Capacitor_SMD:C_0603_1608Metric -> Capacitor_SMD:C_1206_3216Metric_Pad1.33x1.80mm_HandSolder; infineonRef (none) -> CFDC; property_1 (none) -> X7R; property_2 (none) -> 25V
- C35: renamed from CGD0N1; footprint Capacitor_SMD:C_0603_1608Metric -> Capacitor_SMD:C_1206_3216Metric_Pad1.33x1.80mm_HandSolder; infineonRef (none) -> CGD0N1; property_1 (none) -> X5R; property_2 (none) -> 50V
- C36: renamed from CGD0N2; footprint Capacitor_SMD:C_0603_1608Metric -> Capacitor_SMD:C_1206_3216Metric_Pad1.33x1.80mm_HandSolder; infineonRef (none) -> CGD0N0; property_1 (none) -> X7R; property_2 (none) -> 50V
- C37: renamed from CVGDC1; footprint Capacitor_SMD:C_1206_3216Metric -> Capacitor_SMD:C_1206_3216Metric_Pad1.33x1.80mm_HandSolder; infineonRef (none) -> CVGDC; property_1 (none) -> X7R; property_2 (none) -> 25V
- C38: renamed from CGD2; footprint Capacitor_SMD:C_0603_1608Metric -> Capacitor_SMD:C_1206_3216Metric_Pad1.33x1.80mm_HandSolder; infineonRef (none) -> CGD1; property_1 (none) -> X7R; property_2 (none) -> 25V
- C39: renamed from CCDC1; footprint Capacitor_SMD:C_0603_1608Metric -> Capacitor_SMD:C_1206_3216Metric_Pad1.33x1.80mm_HandSolder; infineonRef (none) -> CCDC; property_1 (none) -> X7R; property_2 (none) -> 25V
- C4: renamed from CPVDD0A1; footprint Capacitor_SMD:C_1206_3216Metric -> Capacitor_SMD:C_1206_3216Metric_Pad1.33x1.80mm_HandSolder; infineonRef (none) -> CPVDD0A; property_1 (none) -> X7R; property_2 (none) -> 50V
- C40: renamed from CFGD1; footprint Capacitor_SMD:C_0603_1608Metric -> Capacitor_SMD:C_1206_3216Metric_Pad1.33x1.80mm_HandSolder; infineonRef (none) -> CFGD; property_1 (none) -> X7R; property_2 (none) -> 50V
- C41: renamed from CCREF1; footprint Capacitor_SMD:C_0603_1608Metric -> Capacitor_SMD:C_1206_3216Metric_Pad1.33x1.80mm_HandSolder; infineonRef (none) -> CCREF; property_1 (none) -> X7R; property_2 (none) -> 25V
- C43: renamed from CAPIN0B1; footprint Capacitor_SMD:C_0603_1608Metric -> Capacitor_SMD:C_1206_3216Metric_Pad1.33x1.80mm_HandSolder; infineonRef (none) -> CAPIN0B; property_1 (none) -> X5R; property_2 (none) -> 10V
- C44: renamed from CAPIN0A1; footprint Capacitor_SMD:C_0603_1608Metric -> Capacitor_SMD:C_1206_3216Metric_Pad1.33x1.80mm_HandSolder; infineonRef (none) -> CAPIN0A; property_1 (none) -> X5R; property_2 (none) -> 10V
- C45: renamed from CAPIN1B1; footprint Capacitor_SMD:C_0603_1608Metric -> Capacitor_SMD:C_1206_3216Metric_Pad1.33x1.80mm_HandSolder; infineonRef (none) -> CAPIN1B; property_1 (none) -> X5R; property_2 (none) -> 10V
- C46: renamed from CAPIN1A1; footprint Capacitor_SMD:C_0603_1608Metric -> Capacitor_SMD:C_1206_3216Metric_Pad1.33x1.80mm_HandSolder; infineonRef (none) -> CAPIN1A; property_1 (none) -> X5R; property_2 (none) -> 10V
- C5: renamed from CPVDD1A1; footprint Capacitor_SMD:C_1206_3216Metric -> Capacitor_SMD:C_1206_3216Metric_Pad1.33x1.80mm_HandSolder; infineonRef (none) -> CPVDD1A; property_1 (none) -> X7R; property_2 (none) -> 50V
- C6: renamed from CPVDD1B1; footprint Capacitor_SMD:C_0603_1608Metric -> Capacitor_SMD:C_1206_3216Metric_Pad1.33x1.80mm_HandSolder; infineonRef (none) -> CPVDD1B; property_1 (none) -> X5R; property_2 (none) -> 50V
- C7: renamed from CPVDD0B2; footprint Capacitor_SMD:C_0603_1608Metric -> Capacitor_SMD:C_1206_3216Metric_Pad1.33x1.80mm_HandSolder; infineonRef (none) -> CAVDD0; property_1 (none) -> X7R; property_2 (none) -> 25V
- C8: renamed from C1; footprint Capacitor_THT:C_Rect_L13.0mm_W5.0mm_P10.00mm_FKS3_FKP3_MKS4 -> Capacitor_TH_TDK:C_Rect_L7.3_W4.5_P5.0; infineonRef (none) -> C0A0; property_1 (none) -> L13.0xW5.0
- C9: renamed from C5; footprint Capacitor_THT:C_Rect_L7.2mm_W4.5mm_P5.00mm_FKS2_FKP2_MKS2_MKP2 -> Capacitor_TH_TDK:C_Rect_L7.3_W4.5_P5.0; infineonRef (none) -> C0B1; property_1 (none) -> L7.2xW4.5
- CIN1: value 22nF -> 0.022uF; footprint Capacitor_SMD:C_0603_1608Metric -> Capacitor_SMD:C_1206_3216Metric_Pad1.33x1.80mm_HandSolder; infineonRef (none) -> CIN0; property_1 (none) -> X7R; property_2 (none) -> 50V
- CIN2: value 22nF -> 0.022uF; footprint Capacitor_SMD:C_0603_1608Metric -> Capacitor_SMD:C_1206_3216Metric_Pad1.33x1.80mm_HandSolder; infineonRef (none) -> CIN1; property_1 (none) -> X7R; property_2 (none) -> 50V
- CONN3: renamed from PCTRL1; infineonRef (none) -> PCTRL1
- CONN4: renamed from PAUDIO1; infineonRef (none) -> PAUDIO1
- L1: renamed from LSUP1; value Ferrite 2743019447 -> 47; infineonRef (none) -> LSUP1
- L2: renamed from L1; value 3.3uH -> 6.8uH; footprint Inductor_SMD:L_Bourns_SRP1245A -> Inductor_TH_Bourns:L_Radia_Zylinder_D9.0_P5.0
- L3: value 3.3uH -> 10uH; footprint Inductor_SMD:L_Bourns_SRP1245A -> Inductor_TH_Bourns:RLB0712-100KL
- L4: renamed from L2; value 3.3uH -> 6.8uH; footprint Inductor_SMD:L_Bourns_SRP1245A -> Inductor_TH_Bourns:L_Radia_Zylinder_D9.0_P5.0
- LED1: renamed from CLIP_LED_1; footprint LED_SMD:LED_1206_3216Metric -> LED_SMD:LED_1206_3216Metric_Pad1.42x1.75mm_HandSolder; infineonRef (none) -> CLIP_LED_1
- LED2: renamed from ERROR_LED_1; footprint LED_SMD:LED_1206_3216Metric -> LED_SMD:LED_1206_3216Metric_Pad1.42x1.75mm_HandSolder; infineonRef (none) -> ERROR_LED_1
- R1: renamed from RPVDD1; footprint Resistor_SMD:R_1206_3216Metric -> Resistor_SMD:R_1206_3216Metric_Pad1.30x1.75mm_HandSolder; infineonRef (none) -> RPVDD1
- R2: renamed from R1; footprint Resistor_SMD:R_0603_1608Metric -> Resistor_SMD:R_1206_3216Metric_Pad1.30x1.75mm_HandSolder
- R3: value 3.6 -> 4.7k; footprint Resistor_SMD:R_0603_1608Metric -> Resistor_SMD:R_1206_3216Metric_Pad1.30x1.75mm_HandSolder
- R4: renamed from R2; footprint Resistor_SMD:R_0603_1608Metric -> Resistor_SMD:R_1206_3216Metric_Pad1.30x1.75mm_HandSolder
- R6: renamed from RCLIP_LED_1; footprint Resistor_SMD:R_1206_3216Metric -> Resistor_SMD:R_1206_3216Metric_Pad1.30x1.75mm_HandSolder; infineonRef (none) -> R_CLIP
- R8: renamed from RCLIP_ERROR_1; footprint Resistor_SMD:R_1206_3216Metric -> Resistor_SMD:R_1206_3216Metric_Pad1.30x1.75mm_HandSolder; infineonRef (none) -> R_ERROR
- renumbered J1 to CONN1, J2 to CONN2
Connections:
- net AD0: now also JP5.2 (C)
- net AD1: now also JP9.2 (C)
- net ENABLE: now also JP2.2 (B)
- net GND: now also C8.2, C15.2, C16.2, C19.2, C20.2, C23.2, C24.1, C27.2, C28.2, JP2.1 (A), JP3.1 (A), JP5.1 (A), JP6.1 (A), JP7.1 (A), JP9.1 (A), U1.4 (PGND), U1.5 (AGND), U1.EPAD (EP); no longer C8.1
- net MUTE: now also JP4.2 (B)
- net OUT1A: now also L5.2; no longer L3.2
- net OUT1B: now also L6.2
- net PVDD: now also C15.1, C16.1, U1.10 (EN), U1.2 (SUP)
- net VDD: now also R3.1, JP1.2 (C), JP3.3 (B), JP4.1 (A), JP5.3 (B), JP9.3 (B)
- net at R3.2: now also U1.6 (*RESET)
- net at CONN2.1 (Pin_1): now also C9.2, L2.1, R2.1
- net at R2.2: now also C8.1; no longer C8.2
- net at C13.1, L4.1, R4.2: now also CONN2.2 (Pin_2); no longer CONN2.3 (Pin_3)
- net at C44.1, CONN4.2 (Pin_2): now also JP6.2 (B)
- net at C45.1, CONN4.5 (Pin_5): now also JP7.2 (B), JP8.2 (B)
- net CLK renamed CLKIO
- net CLKIO: now also JP8.1 (A)
- net CLKM/S renamed CLKMS
- net CLKMS: now also JP3.2 (C)
- net ERROR renamed ERR
- net SCLK renamed IN0A
- net SD0 renamed IN1A
- net SD1 renamed IN1B
- net WS renamed IN0B
- new net: C24.2, CONN2.3 (Pin_3), L5.1, R5.1
- new net: C28.1, CONN2.4 (Pin_4), L6.1, R7.2
- new net: C19.1, U1.7 (MODE), U1.8 (BIAS)
- new net: C14.2, L3.1, U1.3 (LX)
- new net: C14.1, U1.1 (BST)
- new net: C27.1, R7.1
- new net: C23.1, R5.2
- new net Buck_5V: JP1.1 (A)
- new net IC_5V: C20.1, JP1.3 (B), L3.2, U1.9 (OUT)
Other:
- moved on the sheet: C12, C13, C3, C32, C33, C34, C4, C5, C6, C7, C8, C9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
