File: ma12070p_amp_v07.kicad_pcb (KiCad board)
At the start: 2 copper layers, 100.4 x 80.4 mm, 83 parts, among them U1 MAX16956, U2 MA12070P

Commit message: DRC Check
Routing:
- net VDD: track 185.7 -> 191.1 mm
- net Net-(C43-Pad1): track 47.7 -> 45.8 mm
- net Net-(C21-Pad1): track 9.75 -> 8.63 mm
- net ERR: track 42.3 -> 41.3 mm
- net CLIP: track 41.7 -> 41.0 mm
- net GND: vias 201 -> 200
