File: ma12070p_amp_v06.kicad_sch (KiCad schematic)
At the start: 83 parts, among them U1 MAX16956, U2 MA12070P

Commit message: added kicad logo to board
Changed lines of the file:
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@@
     (pin "2")
+  )
+  (symbol (lib_id "logo:LOGO") (at 356.235 21.59 0) (unit 1)
+    (in_bom yes) (on_board yes) (fields_autoplaced)
+    (property "Reference" "#G1" (id 0) (at 356.235 0.127 0)
+      (effects (font (size 1.27 1.27)) hide)
+    )
+    (property "Value" "LOGO" (id 1) (at 356.235 43.053 0)
+      (effects (font (size 1.27 1.27)) hide)
+    )
+    (property "Footprint" "logo:logo" (id 2) (at 356.235 21.59 0)
+      (effects (font (size 1.27 1.27)) hide)
+    )
+    (property "Datasheet" "" (id 3) (at 356.235 21.59 0)
+      (effects (font (size 1.27 1.27)) hide)
+    )
   )
   (symbol (lib_id "power:PWR_FLAG") (at 132.715 153.67 0) (unit 1)
@@
       (reference "#FLG07") (unit 1) (value "PWR_FLAG") (footprint "")
     )
+    (path "/d8d04eb0-7ed8-4205-bb00-15d7a4a02a43"
+      (reference "#G1") (unit 1) (value "LOGO") (footprint "logo:logo")
+    )
     (path "/00000000-0000-0000-0000-0000603ae9e1"

Commit message: working on v0.7
Parts:
- added JP9: SolderJumper_3_Open, Jumper:SolderJumper-3_P1.3mm_Open_Pad1.0x1.5mm, symbol Jumper:SolderJumper_3_Open
- JP1: footprint Jumper:SolderJumper-3_P1.3mm_Open_Pad1.0x1.5mm -> Connector_PinHeader_2.54mm:PinHeader_1x03_P2.54mm_Vertical; symbol Jumper:SolderJumper_3_Open -> Jumper:Jumper_3_Open
- JP10, JP4: value SolderJumper_3_Open -> Jumper:Jumper_3_Open; footprint Jumper:SolderJumper-3_P1.3mm_Open_Pad1.0x1.5mm -> Connector_PinHeader_2.54mm:PinHeader_1x03_P2.54mm_Vertical; symbol Jumper:SolderJumper_3_Open -> Jumper:Jumper_3_Open
- JP11: renamed from JP9; footprint Jumper:SolderJumper-3_P1.3mm_Open_Pad1.0x1.5mm -> Connector_PinHeader_2.54mm:PinHeader_1x03_P2.54mm_Vertical; symbol Jumper:SolderJumper_3_Open -> Jumper:Jumper_3_Open
- JP2, JP3, JP6, JP7, JP8: footprint Jumper:SolderJumper-2_P1.3mm_Open_Pad1.0x1.5mm -> Connector_PinHeader_2.54mm:PinHeader_1x02_P2.54mm_Vertical; symbol Jumper:SolderJumper_2_Open -> Jumper:Jumper_2_Open
Connections:
- net CLKIO: now also JP8.2 (B); no longer JP8.1 (A)
- net GND: now also JP6.2 (B), JP7.2 (B), JP9.1 (A); no longer JP6.1 (A), JP7.1 (A), U2.50 (MSEL1)
- net IN0A: now also C41.1, CONN5.1 (Pin_1)
- net IN0B: now also C42.1, CONN5.2 (Pin_2), JP6.1 (A)
- net IN1A: now also C44.2, CONN5.4 (Pin_4)
- net IN1B: now also C43.1, CONN5.5 (Pin_5), JP7.1 (A), JP8.1 (A)
- net VDD: now also JP9.3 (B); no longer JP4.3 (B)
- net VSUP: now reaches CONN1.1 (Pin_1), R1.1
- net CF0AP: now reaches C10.1, C11.1, U2.6 (CF0AP)
- net CF0AN: now reaches C10.2, C11.2, U2.3 (CF0AN)
- net CF0BP: now reaches C17.1, C18.1, U2.9 (CF0BP)
- net CF0BN: now reaches C17.2, C18.2, U2.12 (CF0BN)
- net CF1AP: now reaches C21.1, C22.1, U2.43 (CF1AP)
- net CF1AN: now reaches C21.2, C22.2, U2.46 (CF1AN)
- net CF1BP: now reaches C26.1, C27.1, U2.40 (CF1BP)
- net CF1BN: now reaches C26.2, C27.2, U2.37 (CF1BN)
- net CGD1N: now reaches C30.1, C31.1, C32.2, U2.52 (CGD1N)
- net CGD1P: now reaches C30.2, U2.53 (CGD1P)
- net VGDC: now reaches C34.2, U2.54 (VGDC)
- net CDC: now reaches C38.1, U2.56 (CDC)
- net CREF: now reaches C40.1, U2.20 (CREF)
- net CFGDN: now reaches C39.1, U2.63 (CFGDN)
- net CFGDP: now reaches C39.2, U2.62 (CFGDP)
- net CFD0P: now reaches C35.1, C36.1, C37.2, U2.60 (CGD0P)
- net CGDON: now reaches C35.2, U2.61 (CGD0N)
- net CFDCP: now reaches C33.1, U2.57 (CFDCP)
- net CFDCN: now reaches C33.2, U2.58 (CFDCN)
- net RCSUP: now reaches CIN1.2, L1.1, R1.2
- net BIAS/MODE: now reaches C19.1, U1.7 (MODE), U1.8 (BIAS)
- net NRST: now reaches R3.2, U1.6 (*RESET)
- net LX: now reaches C14.2, L3.1, U1.3 (LX)
- net BST: now reaches C14.1, U1.1 (BST)
- new net MSEL1: JP9.2 (C), U2.50 (MSEL1)

Commit message: changes
Parts:
- removed JP6, JP7: SolderJumper_2_Open, Connector_PinHeader_2.54mm:PinHeader_1x02_P2.54mm_Vertical, symbol Jumper:Jumper_2_Open
- added R? (x2): 10K, Resistor_SMD:R_1206_3216Metric, symbol Device:R
- C15: value 4,7uF -> 10uF; manufacturerRef (none) -> GRM31CR71E106KA12L
Connections:
- net GND: now also R?.1, R?.2
- net IN0B: now also R?.1
- net IN1B: now also R?.2
Changed lines of the file:
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@@
     (stroke (width 0) (type default) (color 0 0 0 0))
   )
-  (wire (pts (xy 35.56 179.705) (xy 35.56 183.515))
+  (wire (pts (xy 35.56 177.165) (xy 35.56 180.975))
     (stroke (width 0) (type default) (color 0 0 0 0))
   )
@@
     (stroke (width 0) (type default) (color 0 0 0 0))
   )
+  (wire (pts (xy 66.675 160.655) (xy 69.215 160.655))
+    (stroke (width 0) (type default) (color 0 0 0 0))
+  )
   (wire (pts (xy 45.72 179.705) (xy 45.72 184.785))
     (stroke (width 0) (type default) (color 0 0 0 0))
@@
     (pin "2")
   )
-  (symbol (lib_id "Jumper:Jumper_2_Open") (at 35.56 174.625 90) (mirror x) (unit 1)
-    (in_bom yes) (on_board yes)
-    (property "Reference" "JP7" (id 0) (at 29.845 174.625 90)
-      (effects (font (size 1.27 1.27)) (justify right))
-    )
-    (property "Value" "SolderJumper_2_Open" (id 1) (at 32.385 180.34 0)
-      (effects (font (size 1.27 1.27)) (justify right) hide)
-    )
-    (property "Footprint" "Connector_PinHeader_2.54mm:PinHeader_1x02_P2.54mm_Vertical" (id 2) (at 35.56 174.625 0)
-      (effects (font (size 1.27 1.27)) hide)
-    )
-    (property "Datasheet" "~" (id 3) (at 35.56 174.625 0)
-      (effects (font (size 1.27 1.27)) hide)
-    )
-    (pin "1")
-    (pin "2")
-  )
   (symbol (lib_id "Jumper:Jumper_3_Open") (at 96.52 182.245 90) (unit 1)
     (in_bom yes) (on_board yes) (fields_autoplaced)
@@
     (pin "3")
   )
+  (symbol (lib_id "Device:R") (at 62.865 160.655 90) (unit 1)
+    (in_bom yes) (on_board yes)
+    (property "Reference" "R?" (id 0) (at 62.865 156.21 90))
+    (property "Value" "10K" (id 1) (at 62.865 158.115 90))
+    (property "Footprint" "Resistor_SMD:R_1206_3216Metric" (id 2) (at 62.865 162.433 90)
+      (effects (font (size 1.27 1.27)) hide)
+    )
+    (property "Datasheet" "~" (id 3) (at 62.865 160.655 0)
+      (effects (font (size 1.27 1.27)) hide)
+    )
+    (pin "1")
+    (pin "2")
+  )
   (symbol (lib_id "power:PWR_FLAG") (at 102.235 153.67 0) (unit 1)
     (in_bom yes) (on_board yes)
@@
     (pin "1")
   )
-  (symbol (lib_id "power:GND") (at 35.56 183.515 0) (unit 1)
+  (symbol (lib_id "power:GND") (at 35.56 180.975 0) (unit 1)
     (in_bom yes) (on_board yes) (fields_autoplaced)
-    (property "Reference" "#PWR038" (id 0) (at 35.56 189.865 0)
+    (property "Reference" "#PWR038" (id 0) (at 35.56 187.325 0)
       (effects (font (size 1.27 1.27)) hide)
     )
-    (property "Value" "GND" (id 1) (at 35.56 187.96 0))
-    (property "Footprint" "" (id 2) (at 35.56 183.515 0)
+    (property "Value" "GND" (id 1) (at 35.56 185.42 0))
+    (property "Footprint" "" (id 2) (at 35.56 180.975 0)
       (effects (font (size 1.27 1.27)) hide)
     )
-    (property "Datasheet" "" (id 3) (at 35.56 183.515 0)
+    (property "Datasheet" "" (id 3) (at 35.56 180.975 0)
       (effects (font (size 1.27 1.27)) hide)
     )
@@
       (effects (font (size 1.27 1.27)) (justify left))
     )
-    (property "Value" "4,7uF" (id 1) (at 34.925 51.435 0)
+    (property "Value" "10uF" (id 1) (at 34.925 51.435 0)
       (effects (font (size 1.27 1.27)) (justify left))
     )
@@
       (effects (font (size 1.27 1.27)) hide)
     )
+    (property "manufacturerRef" "GRM31CR71E106KA12L" (id 4) (at 31.75 50.8 0)
+      (effects (font (size 1.27 1.27)) hide)
+    )
     (pin "1")
     (pin "2")
@@
     (pin "3")
   )
+  (symbol (lib_id "Device:R") (at 35.56 173.355 180) (unit 1)
+    (in_bom yes) (on_board yes)
+    (property "Reference" "R?" (id 0) (at 31.115 172.72 0)
+      (effects (font (size 1.27 1.27)) (justify right))
+    )
+    (property "Value" "10K" (id 1) (at 30.48 175.26 0)
+      (effects (font (size 1.27 1.27)) (justify right))
+    )
+    (property "Footprint" "Resistor_SMD:R_1206_3216Metric" (id 2) (at 37.338 173.355 90)
+      (effects (font (size 1.27 1.27)) hide)
+    )
+    (property "Datasheet" "~" (id 3) (at 35.56 173.355 0)
+      (effects (font (size 1.27 1.27)) hide)
+    )
+    (pin "1")
+    (pin "2")
+  )
   (symbol (lib_id "power:GND") (at 149.225 186.69 0) (unit 1)
     (in_bom yes) (on_board yes)
@@
     (pin "1")
   )
-  (symbol (lib_id "Jumper:Jumper_2_Open") (at 64.135 160.655 0) (unit 1)
-    (in_bom yes) (on_board yes)
-    (property "Reference" "JP6" (id 0) (at 64.135 158.115 0))
-    (property "Value" "SolderJumper_2_Open" (id 1) (at 63.5 163.195 0)
-      (effects (font (size 1.27 1.27)) hide)
-    )
-    (property "Footprint" "Connector_PinHeader_2.54mm:PinHeader_1x02_P2.54mm_Vertical" (id 2) (at 64.135 160.655 0)
-      (effects (font (size 1.27 1.27)) hide)
-    )
-    (property "Datasheet" "~" (id 3) (at 64.135 160.655 0)
-      (effects (font (size 1.27 1.27)) hide)
-    )
-    (pin "1")
-    (pin "2")
-  )
   (symbol (lib_id "power:PWR_FLAG") (at 157.48 178.435 0) (unit 1)
     (in_bom yes) (on_board yes) (fields_autoplaced)
@@
     )
     (path "/974d82c7-5366-46be-903c-9b0c2aea1d0e"
-      (reference "C15") (unit 1) (value "4,7uF") (footprint "Capacitor_SMD:C_1206_3216Metric")
+      (reference "C15") (unit 1) (value "10uF") (footprint "Capacitor_SMD:C_1206_3216Metric")
     )
     (path "/f9915c62-7e50-4952-8c97-fe955e65aac3"
@@
       (reference "JP5") (unit 1) (value "SolderJumper_3_Open") (footprint "Jumper:SolderJumper-3_P1.3mm_Open_Pad1.0x1.5mm")
     )
-    (path "/e8ff72e8-701d-4ef6-b596-ff6c37c08ea7"
-      (reference "JP6") (unit 1) (value "SolderJumper_2_Open") (footprint "Connector_PinHeader_2.54mm:PinHeader_1x02_P2.54mm_Vertical")
-    )
-    (path "/0f576e76-3559-4fcb-a8b4-e7c2a29d925c"
-      (reference "JP7") (unit 1) (value "SolderJumper_2_Open") (footprint "Connector_PinHeader_2.54mm:PinHeader_1x02_P2.54mm_Vertical")
-    )
     (path "/0c027afe-b5d5-4803-80d3-baa193104d48"
       (reference "JP8") (unit 1) (value "SolderJumper_2_Open") (footprint "Connector_PinHeader_2.54mm:PinHeader_1x02_P2.54mm_Vertical")
@@
       (reference "R8") (unit 1) (value "2k") (footprint "Resistor_SMD:R_1206_3216Metric")
     )
+    (path "/512c9b15-ae23-43d3-9fb1-fa396493c001"
+      (reference "R?") (unit 1) (value "10K") (footprint "Resistor_SMD:R_1206_3216Metric")
+    )
+    (path "/d40983b3-4dfe-4f11-a1a4-4dd9df5f5460"
+      (reference "R?") (unit 1) (value "10K") (footprint "Resistor_SMD:R_1206_3216Metric")
+    )
     (path "/be568931-994d-4a64-b4e6-f6775e31820a"
